Commit message: 调整传感器高度

File: akmbot_description/urdf/akmbot.urdf (robot description, URDF)
Before this commit: robot akmbot, 12 links, 11 joints
Joints:
- joint camera_joint: origin xyz=0.36 0.0022137 0.0975 -> xyz=0.36 0.0022137 0.1
- joint lidar_joint: origin xyz=0.25 0 0.12377 -> xyz=0.25 0 0.18
- joint realsense_joint: origin xyz=0.4 0.0038046 0.052021 -> xyz=0.4 0.0038046 0.05

File: akmbot_description/urdf/akmbot.xacro (robot description, xacro)
@@ -243,5 +243,5 @@
         <parent link="base_link" />
         <child link="camera" />
-        <origin xyz="0.36 0.0022137 0.0975" />
+        <origin xyz="0.36 0.0022137 0.1" />
         <axis xyz="0 0 1" />
     </joint>
@@ -271,5 +271,5 @@
         <parent link="base_link" />
         <child link="real_sense" />
-        <origin xyz="0.4 0.0038046 0.052021" />
+        <origin xyz="0.4 0.0038046 0.05" />
         <axis xyz="0 0 1" />
     </joint>
@@ -299,5 +299,5 @@
         <parent link="base_link" />
         <child link="lidar" />
-        <origin xyz="0.25 0 0.12377" />
+        <origin xyz="0.25 0 0.18" />
         <axis xyz="0 0 1" />
     </joint>
